Commit message: second exercise done

File: src/ex2_fanuc/fanuc_description/robot/fanuc.urdf (robot description, URDF)
Before this commit: robot fanuc, 8 links, 7 joints
Joints:
- joint flange: limit lower=-2.967 upper=2.967 effort=12 velocity=2.443 -> (none)
- joint joint1: limit lower=-2.967 upper=2.967 effort=12 velocity=2.443 -> lower=-3.228 upper=3.228 effort=12 velocity=3.141
- joint joint2: limit lower=-2.967 upper=2.967 effort=12 velocity=2.443 -> lower=-2.268 upper=2.268 effort=12 velocity=3.14
- joint joint3: limit lower=-2.967 upper=2.967 effort=12 velocity=2.443 -> lower=-3.996 upper=3.996 effort=12 velocity=3.490
- joint joint4: limit lower=-2.967 upper=2.967 effort=12 velocity=2.443 -> lower=-3.490 upper=3.490 effort=110 velocity=6.108
- joint joint5: limit lower=-2.967 upper=2.967 effort=12 velocity=2.443 -> lower=-2.443 upper=2.443 effort=110 velocity=6.108
- joint joint6: limit lower=-2.967 upper=2.967 effort=12 velocity=2.443 -> lower=-7.85 upper=7.85 effort=60 velocity=6.981
