Commit message: working in progress ex3

File: src/ex2_comau/comau_description/robot/smartsix.xacro (robot description, xacro)
@@ -1,10 +1,7 @@
 <?xml version="1.0" encoding="utf-8"?>
-<!--
-    This URDF uses the Denavit-Hartenberg (DH) conventions to place the reference frames of the joints.
-    It uses offsets to correctly place the visual and collision meshes. The Comau SmartSix meshes are
-    generated such that their reference frames' origins are always placed in a center of rotation.
-    This allows to offset the visual and collision meshes by using only the displacements in the
-    mechanical drawing, without the need for manual (and error-prone) adjustements.
--->
+<!-- This URDF was automatically created by SolidWorks to URDF Exporter! Originally created by Stephen Brawner (brawner@gmail.com)
+     Commit Version: 1.5.1-0-g916b5db  Build Version: 1.5.7152.31018
+     For more information, please see http://wiki.ros.org/sw_urdf_exporter -->
+<!-- The auto-generated URDF has been modified to be compatible with the last versions of MoveIt! and Gazebo -->
 <robot  name="smartsix"  xmlns:xacro="http://www.ros.org/wiki/xacro">
     <!-- ******************** Used for fixing robot to Gazebo 'base_link' ********************-->
@@ -129,5 +126,5 @@
     </link>
     <joint name="joint3" type="revolute">
-        <!--Joint properties-->
+         <!--Joint properties-->
         <origin xyz="0 -0.59 0" rpy="0 0 -1.5708" />
         <parent link="link2" />
@@ -139,5 +136,5 @@
      <!--************************************************LINK 4********************************************-->
     <link name="link4">
-        <!--Link properties-->
+         <!--Link properties-->
         <inertial>
             <origin xyz="-2.2301E-05 0.0024419 -0.28366" rpy="0 0 0" />
@@ -148,5 +145,5 @@
         </inertial>
         <visual>
-            <origin xyz="0 0 0.64707" rpy="0 0 0" />
+            <origin xyz="0 0 0" rpy="0 0 0" />
             <geometry>
                 <mesh filename="package://comau_description/meshes/visual/link4.dae" />
@@ -155,5 +152,5 @@
         </visual>
         <collision>
-            <origin xyz="0 0 0.64707" rpy="0 0 0" />
+            <origin xyz="0 0 0" rpy="0 0 0" />
             <geometry>
                 <mesh filename="package://comau_description/meshes/collision/link4.stl" />
@@ -162,6 +159,6 @@
     </link>
     <joint name="joint4" type="revolute">
-        <!--Joint properties-->
-        <origin xyz="0.13 0 0" rpy="-1.5708 0 0" />
+          <!--Joint properties-->
+        <origin xyz="0.13 0.64707 0" rpy="-1.5708 0 0" />
         <parent link="link3" />
         <child link="link4" />
@@ -172,5 +169,5 @@
     <!--************************************************LINK 5********************************************-->
     <link name="link5">
-        <!--Link properties-->
+         <!--Link properties-->
         <inertial>
             <origin xyz="-7.297E-05 0.020653 0.00074202" rpy="0 0 0" />
@@ -196,5 +193,5 @@
     <joint name="joint5" type="revolute">
         <!--Joint properties-->
-        <origin xyz="0 0 0.64707" rpy="1.5708 0 0" />
+        <origin xyz="0 0 0" rpy="1.5708 0 0" />
         <parent link="link4" />
         <child link="link5" />
@@ -203,7 +200,7 @@
         <dynamics damping="10.0" friction="50.0" />
     </joint>
-    <!--************************************************LINK 6********************************************-->
+     <!--************************************************LINK 6********************************************-->
     <link name="link6">
-        <!--Link properties-->
+         <!--Link properties-->
         <inertial>
             <origin xyz="-0.00066992 3.0689E-05 -0.0074649" rpy="0 0 0" />
@@ -214,5 +211,5 @@
         </inertial>
         <visual>
-            <origin xyz="0 0 0.095" rpy="0 0 0" />
+            <origin xyz="0 0 0" rpy="0 0 0" />
             <geometry>
                 <mesh filename="package://comau_description/meshes/visual/link6.dae" />
@@ -221,5 +218,5 @@
         </visual>
         <collision>
-            <origin xyz="0 0 0.095" rpy="0 0 0" />
+            <origin xyz="0 0 0" rpy="0 0 0" />
             <geometry>
                 <mesh filename="package://comau_description/meshes/collision/link6.stl" />
@@ -228,6 +225,6 @@
     </link>
     <joint name="joint6" type="revolute">
-        <!--Joint properties-->
-        <origin xyz="0 0 0" rpy="-1.5708 0 0" />
+         <!--Joint properties-->
+        <origin xyz="0 0.095 0" rpy="-1.5708 0 0" />
         <parent link="link5" />
         <child link="link6" />
@@ -236,11 +233,3 @@
         <dynamics damping="10.0" friction="50.0" />
     </joint>
-    <!--************************************************FLANGE********************************************-->
-    <link name="flange"/>
-    <joint name="flange" type="fixed">
-        <!--Joint properties-->
-        <origin xyz="0 0 0.095" rpy="0 0 0" />
-        <parent link="link6" />
-        <child link="flange" />
-    </joint>
 </robot>
